Commit message: markers

File: urdf/tracked_robot_dae.urdf.xacro (robot description, xacro)
@@ -3,4 +3,5 @@
   <xacro:property name="PI" value="3.14" />
   <xacro:property name="scalling" value="1.0" />
+  <xacro:property name="scalling_marker" value="0.15" />
   <!-- Gazebo reference -->
   <xacro:property name="mu1" value="0.8" />
@@ -21,4 +22,8 @@
   <xacro:property name="damping" value="0.0" />
   <xacro:property name="friction" value="0.0" />
+  <!-- Base size -->
+  <xacro:property name="x_size_marker" value="1.0" />
+  <xacro:property name="y_size_marker" value="1.0" />
+  <xacro:property name="z_size_marker" value="0.01" />
   <!-- Base size -->
   <xacro:property name="x_size" value="0.32" />
@@ -100,4 +105,26 @@
      <parent link="dummy"/>
      <child link="base_link"/>
+   </joint>
+  <link name="marker_0">
+    <inertial>
+      <mass value="0.001"/>
+      <origin rpy="0 1.5707 1.5707" xyz="0 0 0"/>
+      <inertia ixx="0.001" ixy="0" ixz="0" iyy="0.001" iyz="0" izz="0.001"/>
+    </inertial>
+    <collision name="marker_0">
+      <geometry>
+        <mesh filename="package://tracked_irl/meshes/markers/marker_0.dae" scale="${scalling_marker} ${scalling_marker} ${scalling_marker}"/>
+      </geometry>
+    </collision>
+    <visual name="marker_0">
+      <geometry>
+        <mesh filename="package://tracked_irl/meshes/markers/marker_0.dae" scale="${scalling_marker} ${scalling_marker} ${scalling_marker}"/>
+      </geometry>
+    </visual>
+  </link>
+  <joint name="marker_0" type="fixed">
+    <origin rpy="0 0 3.14" xyz="${-x_size/2 + x_size_marker *  scalling_marker / 2 } 0 ${0.068 + z_size/2+ z_size_marker * scalling_marker + 0.001}"/>
+     <parent link="base_link"/>
+     <child link="marker_0"/>
    </joint>
 <!-- Left side wheels -->

Commit message: launches

File: urdf/tracked_robot_dae.urdf.xacro (robot description, xacro)
@@ -3,5 +3,5 @@
   <xacro:property name="PI" value="3.14" />
   <xacro:property name="scalling" value="1.0" />
-  <xacro:property name="scalling_marker" value="0.15" />
+  <xacro:property name="scalling_marker" value="0.22" />
   <!-- Gazebo reference -->
   <xacro:property name="mu1" value="0.8" />
@@ -82,10 +82,4 @@
       </geometry>
     </collision>
-    <collision name="tracked_robot__collision_kinect">
-      <origin rpy="0 0 0" xyz="0.05  0    0.102"/>
-      <geometry>
-        <box size="0.057 0.06 ${base_height}"/>
-      </geometry>
-    </collision>
     <visual name="tracked_robot__visual">
       <origin rpy="0 0 0" xyz="0   0   ${base_height}"/>
@@ -94,4 +88,10 @@
       </geometry>
     </visual>
+<!--<collision name="tracked_robot__collision_kinect">
+      <origin rpy="0 0 0" xyz="0.05  0    0.102"/>
+      <geometry>
+        <box size="0.057 0.06 ${base_height}"/>
+      </geometry>
+    </collision>
      <visual name="tracked_robot__visual_kinect">
       <origin rpy="0 0 0" xyz="0.05  0    0.102"/>
@@ -99,5 +99,5 @@
         <box size="0.057 0.06 ${base_height}"/>
       </geometry>
-    </visual> <!---->
+    </visual> -->
   </link>
   <joint name="dummy_joint" type="fixed">
@@ -124,5 +124,6 @@
   </link>
   <joint name="marker_0" type="fixed">
-    <origin rpy="0 0 3.14" xyz="${-x_size/2 + x_size_marker *  scalling_marker / 2 } 0 ${0.068 + z_size/2+ z_size_marker * scalling_marker + 0.001}"/>
+<!--{-x_size/2 + x_size_marker *  scalling_marker / 2 }-->
+    <origin rpy="0 0 3.14" xyz="0 0 ${0.068 + z_size/2+ z_size_marker * scalling_marker + 0.03}"/>
      <parent link="base_link"/>
      <child link="marker_0"/>
@@ -583,5 +584,5 @@
     <dynamics damping="${damping}" friction="${friction}"/>
   </joint>
-<!-- KINECT -->
+<!-- KINECT
       <joint name="camera_joint" type="fixed">
         <origin xyz="0.08     0 0.15" rpy="0 0 0"/>
@@ -657,5 +658,5 @@
           </plugin>
         </sensor>
-      </gazebo>
+      </gazebo>-->
 <!-- END Kinect -->
   <gazebo reference="dummy">
